File: rover-pcb/rover-pcb.kicad_pcb (KiCad board)
At the start: 2 copper layers, 70 x 80 mm, 46 parts, among them J1 12V IN, J2 AVR-ISP-6, J3 Conn_01x04, J4 Conn_01x04, J5 Conn_01x04, J6 Conn_01x04, J7 HC-10, Q1 BSS138, Q2 BSS138, U1 L78L33_SOT89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

Commit message: Adding pads for external LEDs.
Parts:
- added J10: LED_3, rover-pcb:SolderWirePad_1x02_SMD_2x4mm, B.Cu at (198.2, 70.1)
- added J11: LED_4, rover-pcb:SolderWirePad_1x02_SMD_2x4mm, B.Cu at (198.1, 104.0)
- added J8: LED_1, rover-pcb:SolderWirePad_1x02_SMD_2x4mm, B.Cu at (133.9, 89.8)
- added J9: LED_2, rover-pcb:SolderWirePad_1x02_SMD_2x4mm, B.Cu at (133.9, 123.7)
Routing:
- net +12V: track 219.8 -> 245.1 mm
- net GND: track 61.1 -> 51.8 mm, vias 22 -> 32
Other:
- board text added: "+ -"
- board text added: "HC-10"
- board text added: "LED"

Commit message: Adding Joystick PCB.
Other:
- board text added: "ISP"
Changed lines of the file:
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@@
   (general
     (thickness 1.6)
-    (drawings 183)
+    (drawings 184)
     (tracks 513)
     (zones 0)
@@
     )
   )
+  (gr_text ISP (at 166.116 112.268) (layer F.SilkS)
+    (effects (font (size 2 2) (thickness 0.2)))
+  )
   (gr_line (start 158.369 69.088) (end 158.369 57.785) (layer F.SilkS) (width 0.12))
